File: Voyager20.kicad_pcb (KiCad board)
At the start: 2 copper layers, 238.1 x 76.2 mm, 131 parts, among them SW1 SW_PUSH, U1 ATMEGA32U2-AU, U2 PRTR5V0U2X, Y1 16MHz

Commit message: Build numpad
Parts:
- removed CR5, CR6, CR7, CR8: 0.1u, Capacitors_SMD:C_0603
- removed D25, D26, D27, D28, D29, D30, D31, D32, D33, D34, D35, D36, D37, D38, D39, D40, D41, D42, D43, D44, D45, D46, D47: SOD-123, Diodes_SMD:D_SOD-123
- removed the G*** at (265.1, 103.2) (x2)
- removed the G*** at (150.8, 69.8)
- removed MX21, MX22, MX23, MX26, MX27, MX28, MX29, MX30, MX31, MX32, MX33, MX34, MX35, MX36, MX37, MX38, MX39, MX40, MX44, MX45, MX46, MX47: MX-1U, MX_Alps_Hybrid:MXOnly-1U-Hotswap
- removed MX24, MX41, MX43: MX-1.25U, MX_Alps_Hybrid:MXOnly-1.25U-Hotswap
- removed MX25: MX-1.5U, MX_Alps_Hybrid:MXOnly-1.5U-Hotswap
- removed MX42: MX-2U, MX_Alps_Hybrid:MXOnly-2U-Hotswap-ReversedStabilizers
- removed RGB1, RGB2, RGB3, RGB4, RGB5, RGB6, RGB7, RGB8: VAL**, WS2812B:WS2812B
- added G***: LOGO, locallib:ai-ring-6mm, F.Cu at (101.6, 87.3)
- added MX-E-1: MX-2U, MX_Alps_Hybrid:MX-2U-ReversedStabilizers, F.Cu at (104.8, 68.3)
- added MX-E-2: MX-2U, MX_Alps_Hybrid:MX-2U-ReversedStabilizers, F.Cu at (104.8, 106.4)
- added MX-E-3: MX-2U, MX_Alps_Hybrid:MX-2U-ReversedStabilizers, F.Cu at (57.1, 115.9)
- added Q1: Q_NPN_BEC, TO_SOT_Packages_SMD:SOT-23, B.Cu at (74.6, 86.5)
- added R10: 1k, Resistors_SMD:R_0805, B.Cu at (96.8, 39.7)
- added R11: 1k, Resistors_SMD:R_0805, B.Cu at (53.2, 64.3)
- added R12: 1k, Resistors_SMD:R_0805, B.Cu at (69.8, 58.7)
- added R13: 1k, Resistors_SMD:R_0805, B.Cu at (92.9, 68.3)
- added R14: 1k, Resistors_SMD:R_0805, B.Cu at (96.0, 68.3)
- added R15: 1k, Resistors_SMD:R_0805, B.Cu at (55.6, 83.3)
- added R16: 1k, Resistors_SMD:R_0805, B.Cu at (58.7, 83.3)
- added R17: 1k, Resistors_SMD:R_0805, B.Cu at (80.2, 83.3)
- added R18: 1k, Resistors_SMD:R_0805, B.Cu at (104.8, 87.3)
- added R19: 1k, Resistors_SMD:R_0805, B.Cu at (55.6, 95.2)
- added R20: 1k, Resistors_SMD:R_0805, B.Cu at (58.7, 95.2)
- added R21: 1k, Resistors_SMD:R_0805, B.Cu at (77.8, 102.4)
- added R22: 1k, Resistors_SMD:R_0805, B.Cu at (74.6, 102.4)
- added R23: 1k, Resistors_SMD:R_0805, B.Cu at (52.4, 119.1)
- added R24: 1k, Resistors_SMD:R_0805, B.Cu at (61.9, 119.1)
- added R25: 1k, Resistors_SMD:R_0805, B.Cu at (77.8, 119.9)
- added R26: 1k, Resistors_SMD:R_0805, B.Cu at (91.3, 119.9)
- added R27: 1k, Resistors_SMD:R_0805, B.Cu at (74.6, 82.5)
- added R7: 1k, Resistors_SMD:R_0805, B.Cu at (47.6, 49.2)
- added R8: 1k, Resistors_SMD:R_0805, B.Cu at (74.6, 45.2)
- added R9: 1k, Resistors_SMD:R_0805, B.Cu at (77.8, 45.2)
- D18, D23, D24, D9: value SOD-123 -> WS2812B; footprint Diodes_SMD:D_SOD-123 -> LEDs:LED_WS2812B-PLCC4
- MX1, MX10, MX11, MX14, MX15, MX16, MX17, MX18, MX19, MX2, MX20, MX3, MX4, MX5, MX6, MX7, MX8, MX9: footprint MX_Alps_Hybrid:MXOnly-1U-Hotswap -> MX_Alps_Hybrid:MX-1U
- MX12: value MX-1.5U -> MX-1U; footprint MX_Alps_Hybrid:MXOnly-1.5U-Hotswap -> MX_Alps_Hybrid:MX-1U
- MX13: value MX-1.25U -> MX-1U; footprint MX_Alps_Hybrid:MXOnly-1.25U-Hotswap -> MX_Alps_Hybrid:MX-1U
- R1, R2, R3, R4, R5, R6: footprint Resistors_SMD:R_0603 -> Resistors_SMD:R_0805
- SW1: value SW_PUSH -> SW_Push; footprint Molex-0548190589:SKQG-1155865 -> random-keyboard-parts:SKQG-1155865
- U1: value ATMEGA32U2-AU -> ATmega32U2-AU
- U2: footprint locallib:SOT143B -> random-keyboard-parts:SOT143B
- moved D24 211.4 mm to (58.7, 102.4)
- moved R4 191.4 mm to (61.9, 42.1), turned to 0 degrees
- moved R6 191.3 mm to (50.8, 39.7), turned to 270 degrees
- moved U2 189.4 mm to (57.1, 39.7)
- moved USB1 188.9 mm to (57.1, 27.0)
- moved R3 186.2 mm to (61.1, 69.8), turned to 0 degrees
- moved R2 185.8 mm to (61.1, 66.7), turned to 180 degrees
- moved CR1 183.6 mm to (58.7, 54.0)
- moved F1 182.5 mm to (52.4, 49.2), turned to 90 degrees
- moved C1 180.4 mm to (74.9, 56.9), turned to 90 degrees
- moved C2 177.9 mm to (77.5, 56.9), turned to 90 degrees
- moved C5 177.9 mm to (71.9, 67.4), turned to 180 degrees
- moved C6 175.8 mm to (71.9, 64.3)
- moved Y1 174.7 mm to (76.2, 61.1), turned to 0 degrees
- moved D12 174.2 mm to (92.9, 73.8)
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Connections:
- D10 pad 1: ROW0 -> ROW2
- D11 pad 1: ROW0 -> ROW2
- D12 pad 1: ROW0 -> ROW2
- D13 pad 1: ROW1 -> ROW2
- D14 pad 1: ROW1 -> ROW3
- D15 pad 1: ROW1 -> ROW3
- D16 pad 1: ROW1 -> ROW3
- D17 pad 1: ROW1 -> ROW3
- D18 pad 1: ROW1 -> +5V
- D19 pad 1: ROW1 -> ROW4
- D20 pad 1: ROW1 -> ROW4
- D21 pad 1: ROW1 -> ROW4
- D22 pad 1: ROW1 -> ROW4
- D23 pad 1: ROW1 -> +5V
- D24 pad 1: ROW1 -> +5V
- D5 pad 1: ROW0 -> ROW1
- D6 pad 1: ROW0 -> ROW1
- D7 pad 1: ROW0 -> ROW1
- D8 pad 1: ROW0 -> ROW1
- D9 pad 1: ROW0 -> +5V
- D9 pad 2: Net-(D9-Pad2) -> Net-(D18-Pad4)
- MX10 pad 1: COL9 -> COL1
- MX10 pad 2: Net-(D10-Pad2) -> Net-(D11-Pad2)
- MX11 pad 1: COL10 -> COL2
- MX11 pad 2: Net-(D11-Pad2) -> Net-(D12-Pad2)
- MX12 pad 1: COL11 -> COL3
- MX12 pad 2: Net-(D12-Pad2) -> Net-(D13-Pad2)
- MX13 pad 2: Net-(D13-Pad2) -> Net-(D14-Pad2)
- MX14 pad 2: Net-(D14-Pad2) -> Net-(D15-Pad2)
- MX15 pad 2: Net-(D15-Pad2) -> Net-(D16-Pad2)
- MX16 pad 2: Net-(D16-Pad2) -> Net-(D17-Pad2)
- MX17 pad 1: COL4 -> COL0
- MX17 pad 2: Net-(D17-Pad2) -> Net-(D19-Pad2)
- MX18 pad 1: COL5 -> COL1
- MX18 pad 2: Net-(D18-Pad2) -> Net-(D20-Pad2)
- MX19 pad 1: COL6 -> COL2
- MX19 pad 2: Net-(D19-Pad2) -> Net-(D21-Pad2)
- MX20 pad 1: COL7 -> COL3
- MX20 pad 2: Net-(D20-Pad2) -> Net-(D22-Pad2)
- MX5 pad 1: COL4 -> COL0
- MX6 pad 1: COL5 -> COL1
- MX7 pad 1: COL6 -> COL2
- MX8 pad 1: COL7 -> COL3
- MX9 pad 1: COL8 -> COL0
- MX9 pad 2: Net-(D9-Pad2) -> Net-(D10-Pad2)
- U1 pad 10: ROW3 -> Net-(U1-Pad10)
- U1 pad 11: COL11 -> Net-(U1-Pad11)
- U1 pad 12: COL10 -> Net-(U1-Pad12)
- U1 pad 14: COL9 -> Net-(U1-Pad14)
- U1 pad 15: COL8 -> Net-(U1-Pad15)
- U1 pad 16: COL7 -> COL3
- U1 pad 17: COL6 -> COL2
- U1 pad 18: COL5 -> Net-(U1-Pad18)
- U1 pad 19: COL4 -> RGBLED
- U1 pad 20: COL3 -> ROW4
- U1 pad 21: COL2 -> Net-(R27-Pad2)
- U1 pad 22: Net-(U1-Pad22) -> ROW3
- U1 pad 23: RGBLED -> ROW2
- U1 pad 9: ROW2 -> Net-(U1-Pad9)
Routing:
- net GND: track 656.4 -> 345.4 mm, vias 22 -> 11
- net LEDGND: track 0.00 -> 308.1 mm, vias 0 -> 10
- net COL4: track 197.3 -> 0.00 mm, vias 4 -> 0
- net ROW3: track 247.8 -> 52.5 mm
- net ROW0: track 278.7 -> 90.9 mm
- net ROW1: track 264.6 -> 83.8 mm
- net COL5: track 177.1 -> 0.00 mm, vias 4 -> 0
- net ROW2: track 232.2 -> 55.4 mm
- net COL1: track 257.9 -> 93.3 mm, vias 4 -> 0
- net COL0: track 278.9 -> 123.3 mm, vias 4 -> 0
- net COL2: track 236.9 -> 83.1 mm, vias 4 -> 0
- net COL7: track 138.2 -> 0.00 mm, vias 4 -> 0
- net COL6: track 134.7 -> 0.00 mm, vias 3 -> 0
- net COL8: track 119.0 -> 0.00 mm, vias 4 -> 0
- net COL3: track 217.6 -> 100.1 mm, vias 4 -> 1
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Other:
- board size 238.1 x 76.2 mm -> 73 x 95.2 mm
- net class Default: trace_width 0.25 -> 0.254
- net class POWER: trace_width 0.635 -> 0.381
- board text added: "20"
- board text added: "VOYAGER"
- board text added: "Voyager20 PCB Rev 1.0 20190126 kb.ai03.me"
- board text removed: "Distributed by Keyhive | 20181128 | Credits to 40percent.club's Gnap"
- board text removed: "RGB1"
- board text removed: "RGB2"
- board text removed: "RGB3"
- board text removed: "RGB4"
- board text removed: "RGB5"
- board text removed: "RGB6"
- board text removed: "RGB7"
- board text removed: "RGB8"
- board text removed: "UT47.2"
- board text removed: "UT47.2 PCB by ai03 Rev 1.0"
