File: Voyager20.kicad_pcb (KiCad board)
At the start: 2 copper layers, 91.5 x 148 mm, 99 parts, among them J1 Conn_01x04, Q1 Q_NPN_BEC, SW1 SW_Push, U1 ATmega32U2-AU, U2 PRTR5V0U2X, Y1 16MHz

Commit message: Major revision
Parts:
- removed the G*** at (111.1, 15.9)
- removed the REF** at (71.4, -15.1)
- removed the REF** at (81.0, -15.1)
- added G***: LOGO, locallib:ai-10-cu, B.Cu at (113.5, -11.1)
- added G***: LOGO, locallib:ai-10-cu, F.Cu at (113.5, -11.1)
- added REF**: CableTie, locallib:CableTie, F.Cu at (80.2, -13.5)
- added REF**: CableTie, locallib:CableTie, F.Cu at (72.2, -13.5)
- moved SW1 58.9 mm to (95.2, 49.2), turned to 0 degrees
- moved F1 36.5 mm to (87.3, 21.4), turned to 90 degrees
- moved U2 36.5 mm to (82.5, 19.1)
- moved Q1 34.5 mm to (67.0, 16.4)
- moved R27 34.5 mm to (67.0, 12.4)
- moved J1 33.0 mm to (72.2, 13.5)
- moved C1 30.3 mm to (41.7, 22.9), turned to 180 degrees
- moved R2 29.5 mm to (76.2, 31.0), turned to 0 degrees
- moved C2 29.5 mm to (41.7, 20.4), turned to 180 degrees
- moved R3 29.2 mm to (76.2, 27.8), turned to 180 degrees
- moved C6 21.6 mm to (50.0, 27.8), turned to 180 degrees
- moved Y1 21.5 mm to (45.9, 21.7), turned to 90 degrees
- moved R1 21.2 mm to (64.9, 26.2), turned to 90 degrees
- moved C4 21.2 mm to (46.0, 16.7), turned to 180 degrees
- moved R5 18.3 mm to (54.8, 10.3), turned to 270 degrees
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Routing:
- net +5V: track 691.3 -> 642.6 mm, vias 5 -> 8
- net Net-(R1-Pad2): track 17.7 -> 58.3 mm, vias 0 -> 2
- net ROW1: track 86.3 -> 125.2 mm
- net GND: track 131.7 -> 167.5 mm, vias 6 -> 5
- net COL1: track 158.1 -> 129.6 mm
- net Net-(R27-Pad2): track 39.5 -> 12.8 mm
- net ROW0: track 82.7 -> 108.9 mm, vias 0 -> 2
- net COL0: track 137.1 -> 159.8 mm, vias 1 -> 2
- net D-: track 7.41 -> 26.1 mm
- net D+: track 7.49 -> 25.2 mm
- net LEDGND: track 395.8 -> 381.8 mm, vias 9 -> 10
- net NLCKLED: track 34.8 -> 47.9 mm
- net ROWFN: track 82.8 -> 70.1 mm, vias 3 -> 2
- net Net-(D26-Pad2): track 6.45 -> 12.8 mm
- net COL2: track 149.0 -> 143.5 mm, vias 3 -> 1
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Other:
- board text added: "1. Strip the USB cable, solder the inner wires to the USB pads on the PCB from the underside 2. Verify correct soldering order for wires; test connectivity 3. Secure the cable's sheathed portion to the PCB via zip ties 4. Solder either the backlight or indicator jumper for num lock LED position"
- board text added: "20-3700"
- board text added: "20190205"
- board text added: "BLACK GREEN WHITE RED"
- board text added: "RED WHITE GREEN BLACK"
- board text added: "USB CABLE ANCHOR"
- board text added: "Voyager20-3700 Rev 1.1"
- board text added: "kb.ai03.me"
- board text removed: "3700"
- board text removed: "4 3 2 1"
- board text removed: "Connection Options a) Hardwire USB cable to USB pads. Optionally zip-tie the cable to the pcb using the hole provided for strength. b) Mount a Mini-XLR connector on the PS2 passthrough hole. Wire to the USB pads, following the numbered order."
